Commit message: motion planning for tendon cube with table in scene is complete, motion planning for robotiq gripper is in progress

File: lbr_description/urdf/med14_robotiq_2f/med14_robotiq_2f.xacro (robot description, xacro)
@@ -4,7 +4,8 @@
     <!-- include the lbr med macro -->
     <xacro:include filename="$(find lbr_description)/urdf/med14/med14_description.xacro" />
-    <xacro:include filename="$(find lbr_description)/urdf/med14_tc/tendon_cube_description.xacro" />
-    <xacro:include filename="$(find lbr_description)/urdf/med14_tc/common_properties.xacro" />
-    <xacro:include filename="$(find lbr_description)/urdf/med14_tc/table_description.xacro" />
+    <xacro:include filename="$(find robotiq_description)/urdf/robotiq_2f_140_macro.urdf.xacro" />
+    <xacro:include filename="$(find lbr_description)/urdf/med14_robotiq_2f/robotiq_adapter_description.xacro" />
+    <xacro:include filename="$(find lbr_description)/urdf/med14_robotiq_2f/common_properties.xacro" />
+    <xacro:include filename="$(find lbr_description)/urdf/med14_robotiq_2f/table_description.xacro" />
     <xacro:arg name="robot_name" default="lbr" />
     <xacro:arg name="mode" default="true" />
@@ -12,5 +13,5 @@
         name="system_config_path"
         default="$(find lbr_description)/ros2_control/lbr_system_config.yaml" />
-    <!-- <xacro:arg name="tc_parent" value="$(arg robot_name)_link_ee" /> -->
+    <xacro:arg name="use_fake_hardware" default="true" />
     <!-- KDL requires a link without inertia -->
     <link name="$(arg robot_name)_floating_link" />
@@ -20,13 +21,21 @@
         <child link="$(arg robot_name)_link_0" />
     </joint>
-    <!-- instantiate robot -->
+    <!-- Instantiate robot -->
     <xacro:med14
         robot_name="$(arg robot_name)"
         mode="$(arg mode)"
         system_config_path="$(arg system_config_path)" />
-    <!-- attach tendon cube -->
-    <xacro:tendon_cube_description
+    <!-- Attach adapter -->
+    <xacro:robotiq_adapter_description
         parent_link="$(arg robot_name)_link_ee"
         robot_name="$(arg robot_name)" />
+    <!-- Attach Robotiq gripper -->
+    <xacro:robotiq_gripper
+        name="RobotiqGripperHardwareInterface"
+        prefix="$(arg robot_name)_"
+        parent="$(arg robot_name)_robotiq_adapter_link"
+        use_fake_hardware="$(arg use_fake_hardware)">
+        <origin xyz="0 0 ${0.05}" rpy="0 0 ${pi/2}" />
+    </xacro:robotiq_gripper>
     <!-- attach table to robot base -->
     <xacro:table_description

File: lbr_description/urdf/med14_tc/tendon_cube_description.xacro (robot description, xacro)
@@ -1,5 +1,5 @@
 <?xml version="1.0"?>
-<robot name="my_robot" xmlns:xacro="http://www.ros.org/wiki/xacro">
-    <xacro:include filename="$(find lbr_description)/urdf/med14_tc/common_properties.xacro" />
+<robot name="tendon_cube" xmlns:xacro="http://www.ros.org/wiki/xacro">
+    <!-- <xacro:include filename="$(find lbr_description)/urdf/med14_tc/common_properties.xacro" /> -->
     <xacro:macro name="tendon_cube_description" params="parent_link robot_name">
         <xacro:property name="base_length" value="0.6" />

Commit message: gripper and robot controllers working toegther in sim

File: lbr_description/urdf/med14_robotiq_2f/med14_robotiq_2f.xacro (robot description, xacro)
@@ -1,5 +1,5 @@
 <?xml version="1.0"?>
 <!-- top level -->
-<robot name="med14" xmlns:xacro="http://www.ros.org/wiki/xacro">
+<robot name="med14_robotiq_2f" xmlns:xacro="http://www.ros.org/wiki/xacro">
     <!-- include the lbr med macro -->
     <xacro:include filename="$(find lbr_description)/urdf/med14/med14_description.xacro" />
@@ -36,6 +36,13 @@
         parent="$(arg robot_name)_robotiq_adapter_link"
         use_fake_hardware="$(arg use_fake_hardware)">
-        <origin xyz="0 0 ${0.05}" rpy="0 0 ${pi/2}" />
+        <origin xyz="0 0 0" rpy="0 0 ${pi/2}" />
     </xacro:robotiq_gripper>
+    <!-- Attach Robotiq gripper NO PREFIX-->
+    <!-- <xacro:robotiq_gripper
+        name="RobotiqGripperHardwareInterface"
+        parent="$(arg robot_name)_robotiq_adapter_link"
+        use_fake_hardware="$(arg use_fake_hardware)">
+        <origin xyz="0 0 0" rpy="0 0 ${pi/2}" />
+    </xacro:robotiq_gripper> -->
     <!-- attach table to robot base -->
     <xacro:table_description

File: lbr_description/urdf/med14_robotiq_2f/robotiq_adapter_description.xacro (robot description, xacro)
@@ -1,8 +1,8 @@
 <?xml version="1.0"?>
-<robot name="my_robot" xmlns:xacro="http://www.ros.org/wiki/xacro">
+<robot name="robtiq_adapter" xmlns:xacro="http://www.ros.org/wiki/xacro">
     <!-- <xacro:include filename="$(find lbr_description)/urdf/med14_tc/common_properties.xacro" /> -->
     <xacro:macro name="robotiq_adapter_description" params="parent_link robot_name">
-        <xacro:property name="cylinder_radius" value="0.045" />
-        <xacro:property name="cylinder_height" value="0.05" />
+        <xacro:property name="cylinder_radius" value="0.0375" />
+        <xacro:property name="cylinder_height" value="0.0168" />
         <link name="${robot_name}_robotiq_adapter_link">
             <visual>
@@ -10,5 +10,5 @@
                     <cylinder radius="${cylinder_radius}" length="${cylinder_height}"/>
                 </geometry>
-                <origin xyz="0 0 ${cylinder_height/2}" rpy="0 0 0" />
+                <origin xyz="0 0 ${-cylinder_height/2}" rpy="0 0 0" />
                 <material name="grey" />
             </visual>
@@ -17,5 +17,5 @@
                     <cylinder radius="${cylinder_radius}" length="${cylinder_height}"/>
                 </geometry>
-                <origin xyz="0 0 ${cylinder_height/2}" rpy="0 0 0" />
+                <origin xyz="0 0 ${-cylinder_height/2}" rpy="0 0 0" />
             </collision>
         </link>
@@ -23,5 +23,5 @@
             <parent link="${parent_link}" />
             <child link="${robot_name}_robotiq_adapter_link" />
-            <origin xyz="0 0 0" rpy="0 0 0" />
+            <origin xyz="0 0 ${cylinder_height}" rpy="0 0 0" />
         </joint>
     </xacro:macro>

Commit message: move to pose server and client now working without thread blocking! also virual controllers for robot AND gripper both working together

File: lbr_description/urdf/med14_robotiq_2f/med14_robotiq_2f.xacro (robot description, xacro)
@@ -38,11 +38,4 @@
         <origin xyz="0 0 0" rpy="0 0 ${pi/2}" />
     </xacro:robotiq_gripper>
-    <!-- Attach Robotiq gripper NO PREFIX-->
-    <!-- <xacro:robotiq_gripper
-        name="RobotiqGripperHardwareInterface"
-        parent="$(arg robot_name)_robotiq_adapter_link"
-        use_fake_hardware="$(arg use_fake_hardware)">
-        <origin xyz="0 0 0" rpy="0 0 ${pi/2}" />
-    </xacro:robotiq_gripper> -->
     <!-- attach table to robot base -->
     <xacro:table_description
