Commit message: calibrating table position

File: lbr_description/urdf/med14_gepetto/workspace_table_description.xacro (robot description, xacro)
@@ -48,5 +48,5 @@
             <parent link="${parent_link}" />
             <child link="${robot_name}_workspace_table_link" />
-            <origin xyz="-0.5 0.2 0.125" rpy="0 0 ${pi/2}" />
+            <origin xyz="-0.5 0.16 0.125" rpy="0 0 ${pi/2}" />
         </joint>
     </xacro:macro>

Commit message: Added phase 4 close

File: lbr_description/urdf/med14_gepetto/workspace_table_description.xacro (robot description, xacro)
@@ -48,5 +48,5 @@
             <parent link="${parent_link}" />
             <child link="${robot_name}_workspace_table_link" />
-            <origin xyz="-0.5 0.2 0.125" rpy="0 0 ${pi/2}" />
+            <origin xyz="-0.5 0.2 0.13" rpy="0 0 ${pi/2}" />
         </joint>
     </xacro:macro>
