Commit message: first ICRA demo test

File: lbr_description/urdf/med14_gepetto/gepetto_hand_description.xacro (robot description, xacro)
@@ -2,4 +2,10 @@
 <robot name="gepetto_hand" xmlns:xacro="http://www.ros.org/wiki/xacro">
     <!-- <xacro:include filename="$(find lbr_description)/urdf/med14_gepetto/common_properties.xacro" /> -->
+    <!--
+        The hand's measured mass and centre of mass, written by
+        gepetto_control/payload_id_node. Generated, unlike the mount offset below,
+        which is copied by hand. Empty until the identification has been run.
+    -->
+    <xacro:include filename="$(find lbr_description)/urdf/med14_gepetto/gepetto_payload.xacro" />
     <!--
         The Gepetto tendon-driven hand, as seen by the arm: a single wrist frame at the
@@ -26,9 +32,10 @@
         <!--
             Marker geometry only, so the frame is visible in RViz. Visualizing the hand
-            itself is deliberately out of scope. No <inertial> and no <collision>, matching
-            the robotiq adapter link, so this needs no inertia macro and adds nothing to
-            the collision scene.
+            itself is deliberately out of scope. No <collision>, matching the robotiq
+            adapter link, so this adds nothing to the collision scene. The <inertial> is
+            whatever payload_id_node last measured, and nothing before the first run.
         -->
         <link name="${robot_name}_gepetto_wrist_link">
+            <xacro:gepetto_payload_inertial />
             <visual>
                 <geometry>

File: lbr_description/urdf/med14_gepetto/workspace_table_description.xacro (robot description, xacro)
@@ -48,5 +48,5 @@
             <parent link="${parent_link}" />
             <child link="${robot_name}_workspace_table_link" />
-            <origin xyz="-0.5 0.16 0.125" rpy="0 0 ${pi/2}" />
+            <origin xyz="-0.5 0.2 0.125" rpy="0 0 ${pi/2}" />
         </joint>
     </xacro:macro>

Commit message: calibrating mount

File: lbr_description/urdf/med14_gepetto/gepetto_hand_description.xacro (robot description, xacro)
@@ -18,4 +18,9 @@
         gepetto_core's transform_from_xyz_rpy builds R = Rz(yaw) @ Ry(pitch) @ Rx(roll),
         which is exactly URDF's <origin rpy="roll pitch yaw"> convention.
+        The z here is NOT the raw CAD number: the Onshape fit gives 0.134688 m, and
+        0.139688 m is that value plus a +5 mm real-world calibration correction found on
+        the physical robot. config.py carries the same corrected value; keep the two in
+        step, and re-apply the correction on top of any fresh measurement rather than
+        pasting the raw fit output.
         WARNING: these numbers are copied by hand and nothing here can detect a stale
         value. They were measured 2026-08-18 against the "gepetto_hand / Assembly 1"
@@ -49,5 +54,5 @@
             <parent link="${parent_link}" />
             <child link="${robot_name}_gepetto_wrist_link" />
-            <origin xyz="-0.009490 -0.010641 0.134688"
+            <origin xyz="-0.009490 -0.010641 0.139688"
                     rpy="1.570796 0.174533 -1.570796" />
         </joint>
