Commit message: workinbg on renaming gepetto hand to epfl hand

File: lbr_description/urdf/med14_allegro/med14_allegro.xacro (robot description, xacro)
@@ -7,5 +7,5 @@
     <xacro:include filename="$(find lbr_description)/urdf/med14_allegro/common_properties.xacro" />
     <xacro:include filename="$(find lbr_description)/urdf/med14_allegro/table_description.xacro" />
-    <xacro:include filename="$(find lbr_description)/urdf/med14_gepetto/workspace_table_description.xacro" />
+    <xacro:include filename="$(find lbr_description)/urdf/med14_epfl/workspace_table_description.xacro" />
     <!-- the hand itself lives in the allegro repo, so there is one model shared by this
          mounted setup and by the standalone allegro_hand.launch.py bringup -->

File: lbr_description/urdf/med14_allegro/table_description.xacro (robot description, xacro)
@@ -1,5 +1,5 @@
 <?xml version="1.0"?>
 <robot name="table" xmlns:xacro="http://www.ros.org/wiki/xacro">
-    <!-- <xacro:include filename="$(find lbr_description)/urdf/med14_gepetto/common_properties.xacro" /> -->
+    <!-- <xacro:include filename="$(find lbr_description)/urdf/med14_epfl/common_properties.xacro" /> -->
     <xacro:macro name="table_description" params="parent_link robot_name">
         <xacro:property name="base_length" value="0.92" />

File: lbr_description/urdf/med14_gepetto/gepetto_hand_description.xacro (robot description, xacro)
@@ -1,20 +1,20 @@
 <?xml version="1.0"?>
-<robot name="gepetto_hand" xmlns:xacro="http://www.ros.org/wiki/xacro">
-    <!-- <xacro:include filename="$(find lbr_description)/urdf/med14_gepetto/common_properties.xacro" /> -->
+<robot name="epfl_hand" xmlns:xacro="http://www.ros.org/wiki/xacro">
+    <!-- <xacro:include filename="$(find lbr_description)/urdf/med14_epfl/common_properties.xacro" /> -->
     <!--
         The hand's measured mass and centre of mass, written by
-        gepetto_control/payload_id_node. Generated, unlike the mount offset below,
+        epfl_control/payload_id_node. Generated, unlike the mount offset below,
         which is copied by hand. Empty until the identification has been run.
     -->
-    <xacro:include filename="$(find lbr_description)/urdf/med14_gepetto/gepetto_payload.xacro" />
+    <xacro:include filename="$(find lbr_description)/urdf/med14_epfl/epfl_payload.xacro" />
     <!--
-        The Gepetto tendon-driven hand, as seen by the arm: a single wrist frame at the
+        The epfl tendon-driven hand, as seen by the arm: a single wrist frame at the
         fixed mount offset from the flange. The hand's own morphology (fingers, tendons)
-        is not modelled here - every finger origin in gepetto_core and every solver pose
+        is not modelled here - every finger origin in epfl_hand_core and every solver pose
         in crest-sparse is measured from this wrist frame, so this frame is all the arm
         side needs.
         The origin below is MountConfig.flange_from_wrist_xyz / _rpy from
-        gepetto_core/src/gepetto_core/config.py, copied verbatim. No conversion is needed:
-        gepetto_core's transform_from_xyz_rpy builds R = Rz(yaw) @ Ry(pitch) @ Rx(roll),
+        epfl_hand_core/src/epfl_hand_core/config.py, copied verbatim. No conversion is needed:
+        epfl_hand_core's transform_from_xyz_rpy builds R = Rz(yaw) @ Ry(pitch) @ Rx(roll),
         which is exactly URDF's <origin rpy="roll pitch yaw"> convention.
         The z here is NOT the raw CAD number: the Onshape fit gives 0.134688 m, and
@@ -24,5 +24,5 @@
         pasting the raw fit output.
         WARNING: these numbers are copied by hand and nothing here can detect a stale
-        value. They were measured 2026-08-18 against the "gepetto_hand / Assembly 1"
+        value. They were measured 2026-08-18 against the "epfl_hand / Assembly 1"
         Onshape assembly. After any change to that assembly, to the mounting bracket, or
         to the hand morphology, re-run
@@ -30,8 +30,8 @@
         from crest-sparse/ and copy the numbers over here AND into config.py. The rotation
         is nearly a pair of right angles, so a flipped one still looks plausible - verify
-        with `ros2 run tf2_ros tf2_echo <robot_name>_link_ee <robot_name>_gepetto_wrist_link`
+        with `ros2 run tf2_ros tf2_echo <robot_name>_link_ee <robot_name>_epfl_wrist_link`
         against HandConfig().mount.T_flange_from_wrist().
     -->
-    <xacro:macro name="gepetto_hand_description" params="parent_link robot_name">
+    <xacro:macro name="epfl_hand_description" params="parent_link robot_name">
         <xacro:property name="marker_size" value="0.03" />
         <!--
@@ -41,6 +41,6 @@
             whatever payload_id_node last measured, and nothing before the first run.
         -->
-        <link name="${robot_name}_gepetto_wrist_link">
-            <xacro:gepetto_payload_inertial />
+        <link name="${robot_name}_epfl_wrist_link">
+            <xacro:epfl_payload_inertial />
             <visual>
                 <geometry>
@@ -51,7 +51,7 @@
             </visual>
         </link>
-        <joint name="${robot_name}_gepetto_wrist_joint" type="fixed">
+        <joint name="${robot_name}_epfl_wrist_joint" type="fixed">
             <parent link="${parent_link}" />
-            <child link="${robot_name}_gepetto_wrist_link" />
+            <child link="${robot_name}_epfl_wrist_link" />
             <origin xyz="-0.009490 -0.010641 0.139688"
                     rpy="1.570796 0.174533 -1.570796" />

File: lbr_description/urdf/med14_gepetto/gepetto_payload.xacro (robot description, xacro)
@@ -3,8 +3,8 @@
     <!--
         GENERATED FILE. Do not edit by hand. Written by
-        gepetto_control/payload_id_node on 2026-08-25T16:17:57 from 40 static
+        epfl_control/payload_id_node on 2026-08-25T16:17:57 from 40 static
         torque samples over 40 poses (residual RMS 0.696 Nm,
         condition number 1.3). Re-run the node to regenerate.
-        The origin is the identified centre of mass, expressed in lbr_gepetto_wrist_link.
+        The origin is the identified centre of mass, expressed in lbr_epfl_wrist_link.
         The inertia tensor is NOT identified: static gravity torques carry no
         information about it, so the values below are a small isotropic
@@ -12,5 +12,5 @@
         needs them.
     -->
-    <xacro:macro name="gepetto_payload_inertial">
+    <xacro:macro name="epfl_payload_inertial">
         <inertial>
             <mass value="0.856730" />

File: lbr_description/urdf/med14_gepetto/med14_gepetto.xacro (robot description, xacro)
@@ -1,11 +1,11 @@
 <?xml version="1.0"?>
 <!-- top level -->
-<robot name="med14_gepetto" xmlns:xacro="http://www.ros.org/wiki/xacro">
+<robot name="med14_epfl" xmlns:xacro="http://www.ros.org/wiki/xacro">
     <!-- include the lbr med macro -->
     <xacro:include filename="$(find lbr_description)/urdf/med14/med14_description.xacro" />
-    <xacro:include filename="$(find lbr_description)/urdf/med14_gepetto/gepetto_hand_description.xacro" />
-    <xacro:include filename="$(find lbr_description)/urdf/med14_gepetto/common_properties.xacro" />
-    <xacro:include filename="$(find lbr_description)/urdf/med14_gepetto/table_description.xacro" />
-    <xacro:include filename="$(find lbr_description)/urdf/med14_gepetto/workspace_table_description.xacro" />
+    <xacro:include filename="$(find lbr_description)/urdf/med14_epfl/epfl_hand_description.xacro" />
+    <xacro:include filename="$(find lbr_description)/urdf/med14_epfl/common_properties.xacro" />
+    <xacro:include filename="$(find lbr_description)/urdf/med14_epfl/table_description.xacro" />
+    <xacro:include filename="$(find lbr_description)/urdf/med14_epfl/workspace_table_description.xacro" />
     <xacro:arg name="robot_name" default="lbr" />
     <xacro:arg name="mode" default="true" />
@@ -28,6 +28,6 @@
         mode="$(arg mode)"
         system_config_path="$(arg system_config_path)" />
-    <!-- attach the gepetto hand wrist frame to the flange -->
-    <xacro:gepetto_hand_description
+    <!-- attach the epfl hand wrist frame to the flange -->
+    <xacro:epfl_hand_description
         parent_link="$(arg robot_name)_link_ee"
         robot_name="$(arg robot_name)" />
