Commit message: flipped hand mount

File: lbr_description/urdf/med14_allegro/allegro_mount_description.xacro (robot description, xacro)
@@ -31,5 +31,5 @@
             <parent link="${parent_link}" />
             <child link="${robot_name}_allegro_mount_link" />
-            <origin xyz="0 0 ${mount_height}" rpy="0 0 0" />
+            <origin xyz="0 0 ${mount_height}" rpy="0 0 ${pi}" />
         </joint>
     </xacro:macro>
