Commit message: updated gepetto hand references to epfl hand references

File: lbr_description/urdf/med14_epfl/epfl_hand_description.xacro (robot description, xacro)
@@ -4,6 +4,7 @@
     <!--
         The hand's measured mass and centre of mass, written by
-        epfl_control/payload_id_node. Generated, unlike the mount offset below,
-        which is copied by hand. Empty until the identification has been run.
+        gepetto_control/payload_id_node. Generated, unlike the mount offset below,
+        which is copied by hand. The macro retains its gepetto_ros API name so a
+        regenerated payload file remains compatible with this description.
     -->
     <xacro:include filename="$(find lbr_description)/urdf/med14_epfl/epfl_payload.xacro" />
@@ -42,5 +43,5 @@
         -->
         <link name="${robot_name}_epfl_wrist_link">
-            <xacro:epfl_payload_inertial />
+            <xacro:gepetto_payload_inertial />
             <visual>
                 <geometry>
@@ -57,4 +58,15 @@
                     rpy="1.570796 0.174533 -1.570796" />
         </joint>
+        <!--
+            Compatibility alias for the unchanged gepetto_ros API. Its nodes still
+            resolve <robot_name>_gepetto_wrist_link; new descriptions, planning
+            groups, and integrations should use <robot_name>_epfl_wrist_link.
+        -->
+        <link name="${robot_name}_gepetto_wrist_link" />
+        <joint name="${robot_name}_gepetto_wrist_compat_joint" type="fixed">
+            <parent link="${robot_name}_epfl_wrist_link" />
+            <child link="${robot_name}_gepetto_wrist_link" />
+            <origin xyz="0 0 0" rpy="0 0 0" />
+        </joint>
     </xacro:macro>
 </robot>

File: lbr_description/urdf/med14_epfl/epfl_payload.xacro (robot description, xacro)
@@ -3,5 +3,5 @@
     <!--
         GENERATED FILE. Do not edit by hand. Written by
-        epfl_control/payload_id_node on 2026-08-25T16:17:57 from 40 static
+        gepetto_control/payload_id_node on 2026-08-25T16:17:57 from 40 static
         torque samples over 40 poses (residual RMS 0.696 Nm,
         condition number 1.3). Re-run the node to regenerate.
@@ -12,5 +12,5 @@
         needs them.
     -->
-    <xacro:macro name="epfl_payload_inertial">
+    <xacro:macro name="gepetto_payload_inertial">
         <inertial>
             <mass value="0.856730" />

Commit message: finished updating reference change for epfl hand

File: lbr_description/urdf/med14_epfl/epfl_hand_description.xacro (robot description, xacro)
@@ -4,7 +4,7 @@
     <!--
         The hand's measured mass and centre of mass, written by
-        gepetto_control/payload_id_node. Generated, unlike the mount offset below,
-        which is copied by hand. The macro retains its gepetto_ros API name so a
-        regenerated payload file remains compatible with this description.
+        epfl_hand_control/payload_id_node. Generated, unlike the mount offset below,
+        which is copied by hand. The generated macro name is part of the ROS stack's
+        interface and must remain compatible with this description.
     -->
     <xacro:include filename="$(find lbr_description)/urdf/med14_epfl/epfl_payload.xacro" />
@@ -43,5 +43,5 @@
         -->
         <link name="${robot_name}_epfl_wrist_link">
-            <xacro:gepetto_payload_inertial />
+            <xacro:epfl_payload_inertial />
             <visual>
                 <geometry>
@@ -58,15 +58,4 @@
                     rpy="1.570796 0.174533 -1.570796" />
         </joint>
-        <!--
-            Compatibility alias for the unchanged gepetto_ros API. Its nodes still
-            resolve <robot_name>_gepetto_wrist_link; new descriptions, planning
-            groups, and integrations should use <robot_name>_epfl_wrist_link.
-        -->
-        <link name="${robot_name}_gepetto_wrist_link" />
-        <joint name="${robot_name}_gepetto_wrist_compat_joint" type="fixed">
-            <parent link="${robot_name}_epfl_wrist_link" />
-            <child link="${robot_name}_gepetto_wrist_link" />
-            <origin xyz="0 0 0" rpy="0 0 0" />
-        </joint>
     </xacro:macro>
 </robot>

File: lbr_description/urdf/med14_epfl/epfl_payload.xacro (robot description, xacro)
@@ -3,5 +3,5 @@
     <!--
         GENERATED FILE. Do not edit by hand. Written by
-        gepetto_control/payload_id_node on 2026-08-25T16:17:57 from 40 static
+        epfl_hand_control/payload_id_node on 2026-08-25T16:17:57 from 40 static
         torque samples over 40 poses (residual RMS 0.696 Nm,
         condition number 1.3). Re-run the node to regenerate.
@@ -12,5 +12,5 @@
         needs them.
     -->
-    <xacro:macro name="gepetto_payload_inertial">
+    <xacro:macro name="epfl_payload_inertial">
         <inertial>
             <mass value="0.856730" />
